File: USB_HUB.kicad_sch (KiCad schematic)
At the start: 7 parts, among them U10 SL2.1S, Y1 12M

Commit message: Turn overall Lib to local Lib to avoid incorrect display of schematics
Parts:
- removed U10: SL2.1S, MyLib:SL2.1S-SSOP-16, symbol My_Library:SL2.1S
- added U10: SL2.1S, PcbLib:SL2.1S-SSOP-16, symbol SymLib:SL2.1S
Connections:
- net +5V: now also U10.7 (VDD5)
- net D+: now also U10.6 (UDP)
- net D-: now also U10.5 (UDM)
- net GND: now also U10.8 (VSS)
- net USB0_D+: now also U10.4 (DP1)
- net USB0_D-: now also U10.3 (DM1)
- net USB1_D+: now also U10.2 (DP2)
- net USB1_D-: now also U10.1 (DM2)
- net USB2_D+: now also U10.16 (DP3)
- net USB2_D-: now also U10.15 (DM3)
- net USB3_D+: now also U10.14 (DP4)
- net USB3_D-: now also U10.13 (DM4)
- net XIN: now also U10.12 (XIN)
- net XOUT: now also U10.11 (XOUT)
- net at C38.1: now also U10.10 (VDD18)
- net at C37.1: now also U10.9 (VDD33)
Changed lines of the file:
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@@
     (pin "1")
+  )
+  (symbol (lib_id "SymLib:SL2.1S") (at 141.732 102.362 0) (unit 1)
+    (in_bom yes) (on_board yes) (fields_autoplaced)
+    (property "Reference" "U10" (id 0) (at 142.2274 116.1447 0)
+      (effects (font (size 1.27 1.27)) (justify left))
+    )
+    (property "Value" "SL2.1S" (id 1) (at 142.2274 118.9198 0)
+      (effects (font (size 1.27 1.27)) (justify left))
+    )
+    (property "Footprint" "PcbLib:SL2.1S-SSOP-16" (id 2) (at 140.97 88.519 0)
+      (effects (font (size 1.27 1.27)) hide)
+    )
+    (property "Datasheet" "" (id 3) (at 140.97 88.519 0)
+      (effects (font (size 1.27 1.27)) hide)
+    )
+    (pin "1")
+    (pin "10")
+    (pin "11")
+    (pin "12")
+    (pin "13")
+    (pin "14")
+    (pin "15")
+    (pin "16")
+    (pin "2")
+    (pin "3")
+    (pin "4")
+    (pin "5")
+    (pin "6")
+    (pin "7")
+    (pin "8")
+    (pin "9")
   )
   (symbol (lib_id "power:+5V") (at 113.284 110.49 0) (unit 1)
@@
     (pin "1")
   )
-  (symbol (lib_id "My_Library:SL2.1S") (at 141.732 102.362 0) (unit 1)
-    (in_bom yes) (on_board yes) (fields_autoplaced)
-    (property "Reference" "U10" (id 0) (at 142.2274 116.1447 0)
-      (effects (font (size 1.27 1.27)) (justify left))
-    )
-    (property "Value" "SL2.1S" (id 1) (at 142.2274 118.9198 0)
-      (effects (font (size 1.27 1.27)) (justify left))
-    )
-    (property "Footprint" "MyLib:SL2.1S-SSOP-16" (id 2) (at 140.97 88.519 0)
-      (effects (font (size 1.27 1.27)) hide)
-    )
-    (property "Datasheet" "" (id 3) (at 140.97 88.519 0)
-      (effects (font (size 1.27 1.27)) hide)
-    )
-    (pin "1")
-    (pin "10")
-    (pin "11")
-    (pin "12")
-    (pin "13")
-    (pin "14")
-    (pin "15")
-    (pin "16")
-    (pin "2")
-    (pin "3")
-    (pin "4")
-    (pin "5")
-    (pin "6")
-    (pin "7")
-    (pin "8")
-    (pin "9")
-  )
   (symbol (lib_id "Device:C_Small") (at 113.284 113.538 0) (unit 1)
